File: Rasberry Pi based Cellphone/Main Schematic.sch (EAGLE design)
At the start: 17 parts, among them J1 Main B2B Header, J2 Second B2B Header, J3 Third B2B Header, X1 679105700, X2 679105700, X3 5036-008-210-862, X4 679105700

Commit message: Finished Wiring main b2b connectors
Parts:
- removed USB_POWER_IN: (no value), adafruit:USBMINIB
- added C1: (no value), adafruit:C-USC0402
- added C3: (no value), adafruit:CPOL-USR/2012-12R
- ETHERNET: device con-lemo:EZG-2K-308 -> con-lemo:EZG-1K-310
Connections:
- net N$1 renamed MDI_TRXN3
- net N$2 renamed MDI_TRXP3
- net N$3 renamed MDI_TRXN2
- net N$4 renamed MDI_TRXP2
- net N$5 renamed MDI_TRXN1
- net N$6 renamed MDI_TRXP1
- net N$7 renamed MDI_TRXN0
- net N$8 renamed MDI_TRXP0
- removed net GND: J1.P$11, J1.P$14, J1.P$17, J1.P$2, J1.P$20, J1.P$23, J1.P$26, J1.P$35, J1.P$36, J1.P$5, J1.P$8, J1.P$80
- new net +5V: C3.+, J1.P$71, J1.P$73, J1.P$75, J1.P$77, J1.P$79
- new net 3V2/NVCC_EIM0: J1.P$65, J1.P$67
- new net AUD5_RXD: J2.P$57
- new net AUD5_TXC: J2.P$51
- new net AUD5_TXFS: J2.P$55
- new net BOOT_MODE0: J3.P$3
- new net BOOT_MODE1: J3.P$5
- new net CCM_CLKO1: J2.P$59
- new net CCM_CLKO2: J2.P$63
- new net CLK1_N: J2.P$3
- new net CLK1_P: J2.P$1
- new net CSI_CLK0P: J2.P$13
- new net CSI_D0M: J2.P$8
- new net CSI_D0P: J2.P$10
- new net CSI_D1M: J2.P$14
- new net CSI_D1P: J2.P$16
- new net CSI_D2M: J2.P$20
- new net CSI_D2P: J2.P$22
- new net CSI_D3M: J2.P$26
- new net CSI_D3P: J2.P$28
- new net DI1_D0_CS: J3.P$45
- new net DI1_D1_CS: J3.P$49
- new net DI1_DISP_CLK: J3.P$54
- new net DI1_PIN01: J3.P$53
- new net DI1_PIN02: J3.P$41
- new net DI1_PIN03: J3.P$51
- new net DI1_PIN15: J3.P$43
- new net DISP1_DATA00: J1.P$66
- new net DISP1_DATA01: J1.P$60
- new net DISP1_DATA02: J1.P$56
- new net DISP1_DATA03: J1.P$54
- new net DISP1_DATA04: J1.P$64
- new net DISP1_DATA05: J1.P$62
- new net DISP1_DATA06: J1.P$58
- new net DISP1_DATA07: J3.P$70
- new net DISP1_DATA08: J3.P$55
- new net DISP1_DATA09: J3.P$60
- new net DISP1_DATA10: J3.P$57
- new net DISP1_DATA11: J3.P$68
- new net DISP1_DATA12: J3.P$59
- new net DISP1_DATA13: J3.P$64
- new net DISP1_DATA14: J3.P$63
- new net DISP1_DATA15: J3.P$62
- new net DISP1_DATA16: J3.P$66
- new net DISP1_DATA17: J3.P$69
- new net DISP1_DATA18: J3.P$56
- new net DISP1_DATA19: J3.P$67
- new net DISP1_DATA20: J3.P$58
- new net DISP1_DATA21: J3.P$40
- new net DISP1_DATA22: J3.P$61
- new net DISP1_DATA23: J3.P$65
- new net DSI_CLK0M: J2.P$44
- new net DSI_CLK0P: J2.P$46
- new net DSI_D0M: J2.P$38
- new net DSI_D0P: J2.P$40
- new net DSI_D1M: J2.P$32
- new net DSI_D1P: J2.P$34
- new net ECSPI2_MISO: J1.P$45
- new net ECSPI2_MOSI: J1.P$47
- new net ECSPI2_SCLK: J1.P$49
- new net ECSPI2_SS0: J1.P$32
- new net ECSPI2_SS1: J1.P$34
- new net EIM_WAIT: J3.P$1
- new net ETH_TCT: C1.1, ETHERNET.10, ETHERNET.9, J1.P$29
- new net GNDC: C1.2
- new net HDMI_CLKM: J2.P$39
- new net HDMI_CLKP: J2.P$37
- new net HDMI_D0M: J2.P$33
- new net HDMI_D0P: J2.P$31
- new net HDMI_D1M: J2.P$27
- new net HDMI_D1P: J2.P$25
- new net HDMI_D2M: J2.P$21
- new net HDMI_D2P: J2.P$19
- new net HDMI_HPD: J2.P$49
- new net HDMI_TX_CEC_LINE: J2.P$43
- new net HDMI_TX_DDC_SCL: J2.P$45
- new net HDMI_TX_DDC_SDA: J2.P$47
- new net I2C1_SCL: J1.P$53
- new net I2C1_SDA: J1.P$51
- new net I2C3_SCL: J1.P$31
- new net I2C3_SDA: J1.P$33
- new net LED_10_100_LED_1000: J1.P$25
- new net LED_ACT: J1.P$27
- new net LVDS0_CLK_N: J2.P$78
- new net LVDS0_CLK_P: J2.P$80
- new net LVDS0_TX0_N: J2.P$60
- new net LVDS0_TX0_P: J2.P$62
- new net LVDS0_TX1_N: J2.P$66
- new net LVDS0_TX1_P: J2.P$68
- new net LVDS0_TX2_N: J2.P$72
- new net LVDS0_TX3_N: J2.P$79
- new net LVDS0_TX3_P: J2.P$77
- new net MLB_CN: J3.P$19
- new net MLB_CP: J3.P$17
- new net MLB_DN: J3.P$27
- new net MLB_DP: J3.P$25
- new net MLB_SN: J3.P$23
- new net MLB_SP: J3.P$21
- new net MX6_ONOFF: J3.P$13
- new net NVCC_SD2: J1.P$61
- new net NVCC_SD3: J1.P$63
- new net PCIE_RXM: J2.P$2
- new net PCIE_RXP: J2.P$4
- new net PCIE_TXM: J2.P$7
- new net PCIE_TXP: J2.P$9
- new net PE: C3.-, J1.P$11, J1.P$14, J1.P$17, J1.P$2, J1.P$20, J1.P$23, J1.P$26, J1.P$35, J1.P$36, J1.P$5, J1.P$70, J1.P$72, J1.P$74, J1.P$76, J1.P$78, J1.P$8, J1.P$80, J2.P$11, J2.P$17, J2.P$18, J2.P$23, J2.P$24, J2.P$29, J2.P$30, J2.P$35, J2.P$36, J2.P$48, J2.P$5, J2.P$58, J2.P$6, J2.P$61, J2.P$64, J2.P$70, J2.P$75, J3.P$10, J3.P$16, J3.P$30, J3.P$33, J3.P$47, J3.P$52
- new net PMIC_ON_REQ: J3.P$15
- new net PMIC_STBY_REQ: J3.P$9
- new net POR_B: J2.P$65
- new net PWM1_OUT: J1.P$68
- new net PWM2_OUT: J1.P$41
- new net PWM3_OUT: J1.P$55
- new net PWM4_OUT: J1.P$57
- new net SATA_RXN: J1.P$6
- new net SATA_RXP: J1.P$4
- new net SATA_TXN: J1.P$10
- new net SATA_TXP: J1.P$12
- new net SD2_CD_B: J1.P$50
- new net SD2_CLK: J1.P$38
- new net SD2_CMD: J1.P$40
- new net SD2_DATA0: J1.P$42
- new net SD2_DATA1: J1.P$44
- new net SD2_DATA2: J1.P$46
- new net SD2_DATA3: J1.P$48
- new net SD2_VSELECT: J2.P$73
- new net SD3_CLK: J1.P$37
- new net SD3_CMD: J1.P$39
- new net SD3_DATA0: J3.P$24
- new net SD3_DATA1: J3.P$22
- new net SD3_DATA2: J3.P$20
- new net SD3_DATA3: J3.P$18
- new net SD3_DATA4: J3.P$8
- new net SD3_DATA5: J3.P$6
- new net SD3_DATA6: J3.P$4
- new net SD3_DATA7: J3.P$2
- new net SD3_RST: J3.P$26
- new net SD3_VSELECT: J3.P$28
- new net SD4_CLK: J3.P$32
- new net SD4_CMD: J3.P$34
- new net SD4_DATA0: J3.P$36
- new net SD4_DATA3: J3.P$38
- new net SPDIF_IN: J3.P$35
- new net SPDIF_OUT: J2.P$50
- new net TAMPER: J3.P$7
- new net UART1_RX_DATA: J2.P$54
- new net UART1_TX_DATA: J2.P$52
- new net UART2_CTS_B: J3.P$48
- new net UART2_RTS_B: J3.P$50
- new net UART2_RX_DATA: J3.P$44
- new net UART2_TX_DATA: J3.P$46
- new net UART3_RX_DATA: J3.P$31
- new net UART3_TX_DATA: J3.P$29
- new net USB_H1_OC: J2.P$69
- new net USB_H1_PWR_EN: J1.P$28
- new net USB_H1_VBUS: J1.P$52
- new net USB_HOST_DN: J1.P$24
- new net USB_HOST_DP: J1.P$22
- new net USB_OTG_CHD_B: J2.P$71
- new net USB_OTG_DN: J1.P$18
- new net USB_OTG_DP: J1.P$16
- new net USB_OTG_ID: J2.P$56
- new net USB_OTG_OC: J2.P$67
- new net USB_OTG_PWR_EN: J1.P$30
- new net USB_OTG_VBUS: J1.P$43
- new net VSNVS_3V0: J1.P$69
- new net WDOG1_B: J3.P$42
Other:
- moved on the sheet: EXT_POWER_IN, EXT_RADIO_INTERFACE, GPIOA, GPIOB, HEADSET, J2, J3, MINIDP, U$1, X3

Commit message: Finished Power Supply and Battery Charger
Parts:
- removed MINIDP: 105081-0001, con-molex:105081-0001
- added 5VBOOST: TPS61032-5Vout, texas:TPS61030RSAR
- added BATT: (no value), adafruit:JST_2PIN-SMT-RA
- added BATTERY_CHARGER: MCP73871-2CCI/ML, Microchip_By_element14_Batch_1:MCP73871-2CCI/ML
- added C10, C9: 100uF, adafruit:C-USC0402K
- added C2: 4700uF/10V, adafruit:CPOL-USR/2012-12R
- added C4: 10uF/10V, adafruit:C-USC0402K
- added C5, C6: 10uF, adafruit:C-USC0402K
- added C7: 01uF, adafruit:C-USC0402K
- added C8: 2.2uF, adafruit:C-USC0402K
- added CHRG/LBO: ORANGE, adafruit:LEDCHIP-LED0603
- added D1, D2: (no value), adafruit:DIODESOD-123
- added DONE: GREEN, adafruit:LEDCHIP-LED0603
- added HDMI: 47630-1012, con-molex:47630-1012
- added L1: 6.8uH, rcl:L-USL2825P
- added LT1085: 5v, linear:LT1085
- added ON/OFF?: Potential Location for On Off Switch, adafruit:EG1218S
- added PWR: RED, adafruit:LEDCHIP-LED0603
- added R1: 270K, adafruit:R-US_M0805
- added R10, R3, R4, R5, R8, R9: 1K, adafruit:R-US_M0805
- added R11: 1.87M, adafruit:R-US_M0805
- added R12: 200K, adafruit:R-US_M0805
- added R2, R6: 100K, adafruit:R-US_M0805
- added R7: 2K, adafruit:R-US_M0805
- added RT2: 150K, adafruit:R-US_M0805
- added THERM: 1X2-3.5MM, adafruit:1X2-3.5MM
Connections:
- new net LOWVOLTAGE: 5VBOOST.LBO
- new net N$1: D1.A, EXT_POWER_IN.2
- new net N$10: DONE.A, R4.2
- new net N$11: BATTERY_CHARGER.STAT1/*LBO, CHRG/LBO.C
- new net N$12: BATT.2, BATTERY_CHARGER.VBAT, BATTERY_CHARGER.VBAT_2, BATTERY_CHARGER.VBAT_SENSE, C6.1
- new net N$13: BATTERY_CHARGER.PROG3, R6.2
- new net N$14: BATTERY_CHARGER.PROG1, R7.2
- new net N$15: 5VBOOST.EN, ON/OFF?.P
- new net N$16: BATTERY_CHARGER.THERM, R8.2
- new net N$17: R8.1, RT2.2, THERM.1
- new net N$2: D1.C, LT1085.VIN
- new net N$20: 5VBOOST.LBI, R10.1, R9.2
- new net N$22: 5VBOOST.SW, 5VBOOST.SW_2, L1.2
- new net N$23: 5VBOOST.FB, R11.1, R12.2
- new net N$3: BATTERY_CHARGER.*PG, PWR.C
- new net N$4: D2.A, U$1.VBUS
- new net N$5: BATTERY_CHARGER.VPCC, R1.1, R2.2
- new net N$6: PWR.A, R3.2
- new net N$7: 5VBOOST.VBAT, BATTERY_CHARGER.OUT, BATTERY_CHARGER.OUT_2, C5.1, C7.1, L1.1, ON/OFF?.S, R9.1
- new net N$8: CHRG/LBO.A, R5.2
- new net N$9: BATTERY_CHARGER.STAT2, DONE.C
- new net VIN+5V: 5VBOOST.VOUT, 5VBOOST.VOUT_2, 5VBOOST.VOUT_3, C10.1, C8.1, C9.1, R11.2
- new net VIN+5VBATT: BATTERY_CHARGER.*TE, BATTERY_CHARGER.CE, BATTERY_CHARGER.IN, BATTERY_CHARGER.IN_2, BATTERY_CHARGER.PROG2, BATTERY_CHARGER.SEL, C2.+, C4.1, D2.C, LT1085.VOUT, R1.2, R3.1, R4.1, R5.1
- net PE: now also 5VBOOST.GND, 5VBOOST.PAD, 5VBOOST.PGND, 5VBOOST.PGND_2, 5VBOOST.PGND_3, 5VBOOST.SYNC, BATT.1, BATTERY_CHARGER.EP, BATTERY_CHARGER.VSS, BATTERY_CHARGER.VSS_2, C10.2, C2.-, C4.2, C5.2, C6.2, C7.2, C8.2, C9.2, EXT_POWER_IN.1, LT1085.GND, ON/OFF?.O, R10.2, R12.1, R2.1, R6.1, R7.1, RT2.1, THERM.2, U$1.GND
Other:
- note added: "Need 2x stacked USB or 1x stacked USB and HDMI Reset Button Digital Coax S/PDIF LEDS Various Display connectors (Maybe leave off) RTC battery HEader MIPI CSI connector? 2x Internal USB connections 2x External USB connections"
- note added: "connect 10k thermistor here"
- note added: "connect low voltage to microcontroller to trigger low battery shutdown"
- note removed: "Need 2x stacked USB or 1x stacked USB and Displayport Reset Button Digital Coax S/PDIF LEDS Various Display connectors (Maybe leave off) RTC battery HEader MIPI CSI connector? 2x Internal USB connections 2x External USB connections"
- moved on the sheet: EXT_POWER_IN, HEADSET, U$1

Commit message: added audio, usband some more power stuff
Parts:
- added ADC/DAC: SGTL5000_32QFN, freescale:SGTL5000
- added C11, C12, C13, C18, C23, C24, C25, C28, C29, C30: 0.1uF/16V, adafruit:CPOL-USR/2012-12R
- added C14, C15: 560pF/50V, adafruit:CPOL-USR/2012-12R
- added C16: 10uF/6.3V, adafruit:CPOL-USR/2012-12R
- added C17, C33: 22uF/6.3V, adafruit:CPOL-USR/2012-12R
- added C19, C31, C32, C34, C39, C40, C41, C42: 1uF, adafruit:C-USC0402K
- added C20: 1uF/6.3V, adafruit:CPOL-USR/2012-12R
- added C21, C22: 100uF, adafruit:C-USC0402K
- added C26, C27: 8pF/50V, adafruit:CPOL-USR/2012-12R
- added C35, C36, C37, C38, C43, C44: 10uF, adafruit:CPOL-USR/2012-12R
- added D3: (no value), diode:SCHOTTKY-DIODESMD
- added IC1: PCM2904DB, texas:PCM2904DB
- added L2: 1.5uH, rcl:L-USL2825P
- added L3: BLM15PX121SN1, inductors:BLM15HB121SN1
- added Q1: 20V P-Channel Mosfet, dp_devices:TRANSISTOR_FET_TSM2301CX
- added Q2: (no value), adafruit:CRYSTALCTS406
- added R13: 1K, adafruit:R-US_M0805
- added R14: 73.2K 1%, adafruit:R-US_M0805
- added R15: 24.0K 1%, adafruit:R-US_M0805
- added RESET, SW1, SW2, SW3: SPST_TACT-KMR2, adafruit:SPST_TACT-KMR2
- added RN1: 1.5kΩ, dp_devices:RESISTOR_ARRAY_4
- added RT1, RT3, RT4, RT5, RT6: 2.2K, adafruit:R-US_M0805
- added RT10, RT11: 22Ω, adafruit:R-US_M0805
- added RT12: 1MΩ, adafruit:R-US_M0805
- added RT7: 10K, adafruit:R-US_M0805
- added RT8: 649, adafruit:R-US_M0805
- added RT9: 2.2Ω, adafruit:R-US_M0805
- added SD2_VSELECT: 741G53DCT, 74xx-little-us:741G53DCT
- added U$2: 1V8 Regulator, Microchip_By_element14_Batch_1:MCP1700T-1802E/TT
- added U$3, U$4, U$5: ESD7004, on-semiconductor:ESD7004
- added U1: (no value), cypress:CY7C65632
- added U2: (no value), richtek:RT8070SOP-8
- added U3: (no value), micrel:MIC2026
- added U4, U5, U6: (no value), on-semiconductor:NLX2G16
- added X5, X6: (no value), con-berg:PN87520
- 5VBOOST: value TPS61032-5Vout -> Value
- EXT_RADIO_INTERFACE: value EZG-2K-307 -> EZG-0K-309; device con-lemo:EZG-2K-307 -> con-lemo:EZG-0K-309
Connections:
- net N$7 renamed VBAT
- removed net NVCC_SD3: J1.P$63
- removed net VIN+5V: 5VBOOST.VOUT, 5VBOOST.VOUT_2, 5VBOOST.VOUT_3, C10.1, C8.1, C9.1, R11.2
- removed net VSNVS_3V0: J1.P$69
- new net 3V2/NVCC_EIM2: Q1.S
- new net AUD5_TXD: ADC/DAC.I2S_DIN
- new net HDMI_CEC_C: D3.C, HDMI.P$13, U$5.P$10
- new net HDMI_HPD_C: HDMI.P$19, U$5.P$6
- new net HDMI_SCL_C: HDMI.P$15, U$5.P$9
- new net HDMI_SDA_C: HDMI.P$16, U$5.P$7
- new net MIC_IN: C24.-, HEADSET.2, RT6.1
- new net MUTE/PWR_DOWN: IC1.!SSPND, RN1B.2, RN1C.2, RN1D.2
- new net N$18: ADC/DAC.VDDD, C11.-
- new net N$19: R14.2, R15.1, U2.FB
- new net N$21: ADC/DAC.MIC, C24.+
- new net N$24: ADC/DAC.VAG, C13.-
- new net N$25: C15.+, U2.SS
- new net N$26: D3.A, RT5.1
- new net N$27: R13.1, U2.COMP
- new net N$28: C14.+, R13.2
- new net N$29: ADC/DAC.HP_R, C21.1
- new net N$30: ADC/DAC.HP_L, C22.1
- new net N$31: ADC/DAC.MIC_BIAS, C25.-, RT6.2
- new net N$32: C40.1, IC1.VCCXI
- new net N$33: C41.1, IC1.VCCP2I
- new net N$34: RT8.1, U1.RREF
- new net N$35: RT7.1, U1.GANG
- new net N$36: IC1.VBUS, RT9.1
- new net N$37: IC1.D-, RT11.1
- new net N$38: IC1.D+, RT10.1
- new net N$39: C33.-, U3.GND
- new net N$40: C35.+, IC1.VCCCI
- new net N$41: C36.+, EXT_RADIO_INTERFACE.4, EXT_RADIO_INTERFACE.7, IC1.VCOM
- new net N$42: C42.1, IC1.VCCP1I
- new net N$43: C38.+, IC1.VINL
- new net N$44: C37.+, IC1.VINR
- new net N$45: C38.-, EXT_RADIO_INTERFACE.9
- new net N$46: C37.-, EXT_RADIO_INTERFACE.8
- new net N$47: C43.-, EXT_RADIO_INTERFACE.6
- new net N$48: C44.-, EXT_RADIO_INTERFACE.5
- new net N$49: C43.+, IC1.VOUTR
- new net N$50: C44.+, IC1.VOUTL
- new net N$52: IC1.HID0, SW3.P, SW3.P1
- new net N$53: IC1.HID1, SW2.P, SW2.P1
- new net N$54: RN1B.1, SW1.S, SW1.S1
- new net N$55: IC1.HID2, SW1.P, SW1.P1
- new net N$56: C39.1, IC1.SEL0, IC1.SEL1, IC1.VDDI, RN1A.2
- new net N$57: RN1C.1, SW2.S, SW2.S1
- new net N$58: RN1D.1, SW3.S, SW3.S1
- new net N$7: L2.1, U2.LX
- new net STEREO_OUT_L: C22.2, HEADSET.4
- new net STEREO_OUT_R: C21.2, HEADSET.5
- new net TMDS0+_C: HDMI.P$7, U$4.P$10
- new net TMDS0-_C: HDMI.P$9, U$4.P$9
- new net TMDS1+_C: HDMI.P$4, U$3.P$7
- new net TMDS1-_C: HDMI.P$6, U$3.P$6
- new net TMDS2+_C: HDMI.P$1, U$3.P$10
- new net TMDS2-_C: HDMI.P$3, U$3.P$9
- new net TMDSCLK+_C: HDMI.P$10, U$4.P$7
- new net TMDSCLK-_C: HDMI.P$12, U$4.P$6
- new net USB_HUB_DN1: U1.DD-[1], X6.2
- new net USB_HUB_DN2: U1.DD-[2]
- new net USB_HUB_DN3: U1.DD-[3]
- new net USB_HUB_DN4: RT11.2, U1.DD-[4]
- new net USB_HUB_DP1: U1.DD+[1], X6.3
- new net USB_HUB_DP2: U1.DD+[2]
- new net USB_HUB_DP3: U1.DD+[3]
- new net USB_HUB_DP4: RN1A.1, RT10.2, U1.DD+[4]
- new net VCC_1V8: C18.+, SD2_VSELECTG$1.Y2, U$2.VOUT
- new net V_3V2_FLTR: C28.+, C29.+, C30.+, C31.1, C32.1, L3.2, U1.VCC_A, U1.VCC_A_2, U1.VCC_A_3, U1.VCC_A_4, U1.VCC_A_5, U1.VREG
- new net V_SD: C20.+, MICRO_SD.VDD, Q1.D, RT4.2
- new net XIN: C26.+, IC1.XTI, Q2.1, RT12.1, U1.XIN
- new net XOUT: C27.+, IC1.XTO, Q2.2, RT12.2, U1.XOUT
- net +5V: now also 5VBOOST.VOUT, 5VBOOST.VOUT_2, 5VBOOST.VOUT_3, C10.1, C16.+, C33.+, C34.1, C8.1, C9.1, HDMI.P$18, R11.2, RT9.2, U2.VIN, U3.IN
- net 3V2/NVCC_EIM0: now also ADC/DAC.VDDA, ADC/DAC.VDDIO, C12.-, C17.+, C23.-, J1.P$63, J1.P$69, L2.2, L3.1, R14.1, RT5.2, SD2_VSELECTG$1.Y1, SD2_VSELECTP.VCC, U$2.VIN, U1.SELFPWR, U1.VCC_D, U1.VCC_D_2
- net AUD5_RXD: now also ADC/DAC.I2S_DOUT
- net AUD5_TXC: now also ADC/DAC.I2S_SCLK
- net AUD5_TXFS: now also ADC/DAC.I2S_LRCLK
- net CCM_CLKO1: now also ADC/DAC.SYS_MCLK
- net HDMI_CLKM: now also U$4.P$5
- net HDMI_CLKP: now also U$4.P$4
- net HDMI_D0M: now also U$4.P$2
- net HDMI_D0P: now also U$4.P$1
- net HDMI_D1M: now also U$3.P$5
- net HDMI_D1P: now also U$3.P$4
- net HDMI_D2M: now also U$3.P$2
- net HDMI_D2P: now also U$3.P$1
- net HDMI_HPD: now also U$5.P$5
- net HDMI_TX_CEC_LINE: now also U$5.P$1
- net HDMI_TX_DDC_SCL: now also U$5.P$2
- net HDMI_TX_DDC_SDA: now also U$5.P$4
- net I2C1_SCL: now also ADC/DAC.CTRL_CLK
- net I2C1_SDA: now also ADC/DAC.CTRL_DATA
- net NVCC_SD2: now also C19.1, SD2_VSELECTG$1.COM
- net PE: now also ADC/DAC.AGND, ADC/DAC.CTRL_ADR0_CS, ADC/DAC.CTRL_MODE, ADC/DAC.GND, ADC/DAC.GND2, C11.+, C12.+, C13.+, C14.-, C15.-, C16.-, C17.-, C18.-, C19.2, C20.-, C23.+, C25.+, C26.-, C27.-, C28.-, C29.-, C30.-, C31.2, C32.2, C34.2, C35.-, C36.-, C39.2, C40.2, C41.2, C42.2, HDMI.P$11, HDMI.P$17, HDMI.P$2, HDMI.P$5, HDMI.P$8, HEADSET.1, HEADSET.3, IC1.AGNDC, IC1.AGNDP, IC1.DGND, IC1.DGNDU, IC1.TEST0, MICRO_SD.GND, MICRO_SD.GND1, MICRO_SD.VSS, R15.2, RESET.P1, RT1.2, RT3.1, RT4.1, RT7.2, RT8.2, SD2_VSELECTG$1.INH, SD2_VSELECTP.GND, SD2_VSELECTP.GND@1, U$2.GND, U$3.GND, U$3.GND2, U$4.GND, U$4.GND2, U$5.GND, U$5.GND2, U1.GND, U1.GND_2, U1.GND_3, U1.GND_4, U2.GND, X5.4, X6.4
- net POR_B: now also RESET.S1, U1.RESET#
- net PWM2_OUT: now also Q1.G, RT3.2
- net SD2_CD_B: now also MICRO_SD.CARD_DETECT, MICRO_SD.CARD_DETECT1
- net SD2_CLK: now also MICRO_SD.SCLK
- net SD2_CMD: now also MICRO_SD.DATA_IN
- net SD2_DATA0: now also MICRO_SD.DATA_OUT
- net SD2_DATA1: now also MICRO_SD.DAT1
- net SD2_DATA2: now also MICRO_SD.DAT2
- net SD2_DATA3: now also MICRO_SD.CS
- net SD2_VSELECT: now also RT1.1, SD2_VSELECTG$1.A
- net USB_H1_PWR_EN: now also U3.ENB
- net USB_H1_VBUS: now also U3.OUTB, X6.1
- net USB_HOST_DN: now also U1.D-
- net USB_HOST_DP: now also U1.D+
- net USB_OTG_DN: now also X5.2
- net USB_OTG_DP: now also X5.3
- net USB_OTG_PWR_EN: now also U3.ENA
- net USB_OTG_VBUS: now also U3.OUTA, X5.1
Other:
- note added: "1x stacked USB and HDMI IR? Digital Coax S/PDIF LEDS Various Display connectors (Maybe leave off) RTC battery HEader MIPI CSI connector?"
- note added: "Connect to amplifier if needed"
- note added: "Main Power feeds are +5V and 3V2/NVCC_EIM0"
- note added: "may need amplifiers here"
- note removed: "Need 2x stacked USB or 1x stacked USB and HDMI Reset Button Digital Coax S/PDIF LEDS Various Display connectors (Maybe leave off) RTC battery HEader MIPI CSI connector? 2x Internal USB connections 2x External USB connections"
- moved on the sheet: GPIOA, GPIOB, HDMI, HEADSET

Commit message: random commit
Parts:
- added C45, C46, C47, C48: 10nF/25V, adafruit:C-USC0402
- added C49: (no value), adafruit:CPOL-USR/2012-12R
- added C50: 10uF/6.3V, adafruit:CPOL-USR/2012-12R
- added R16: 10k, adafruit:R-US_M0805
- added R17: 2.2k, adafruit:R-US_M0805
- added U$6: MCP1702T-1502E/CB, Microchip_By_element14_Batch_1:MCP1702T-2502E/CB
Connections:
- removed net 3V2/NVCC_EIM2: Q1.S
- new net MSATA_DISABLE: R16.1, X1-20.S
- new net N$51: C45.1, X1-23.S
- new net N$59: C46.1, X1-25.S
- new net N$60: C47.1, X1-31.S
- new net N$61: C48.1, X1-33.S
- new net V_1V5: C50.+, R17.2, U$6.VOUT, X1-28.S, X1-48.S, X1-6.S
- net 3V2/NVCC_EIM0: now also C49.+, Q1.S, R16.2, U$6.VIN, U1.FIX_PORT4, X1-2.S, X1-24.S, X1-39.S, X1-41.S, X1-52.S
- net I2C1_SCL: now also X1-30.S
- net I2C1_SDA: now also X1-32.S
- net PE: now also C49.-, C50.-, R17.1, U$6.GND, X1-15.S, X1-18.S, X1-21.S, X1-26.S, X1-27.S, X1-29.S, X1-34.S, X1-35.S, X1-37.S, X1-4.S, X1-40.S, X1-43.S, X1-50.S, X1-9.S
- net POR_B: now also X1-22.S
- net SATA_RXN: now also C46.2
- net SATA_RXP: now also C45.2
- net SATA_TXN: now also C47.2
- net SATA_TXP: now also C48.2
Other:
- moved on the sheet: X1-1, X1-10, X1-11, X1-12, X1-13, X1-14, X1-15, X1-16, X1-17, X1-18, X1-19, X1-2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

Commit message: almost finished schematic
Parts:
- removed X2, X4: 679105700, con-molex:679105700
- added C100, C101, C102, C104, C105, C106, C107, C108, C109, C110, C111, C112, C117, C118, C119, C120, C121, C122, C123, C124, C125, C126, C127, C59, C61, C62, C63, C69, C71, C72, C73, C74, C79, C81, C82, C83, C84, C89, C91, C92, C93, C98, C99: 0.1uF, resistor:C-USC0402
- added C103, C113, C114, C115, C116, C60, C67, C70, C75, C78, C80, C85, C88, C90, C94, C95, C96, C97: 0.001uF, resistor:C-USC0402
- added C51, C52: 10uF/6.3V, adafruit:CPOL-USR/2012-12R
- added C53, C54, C55, C56, C57, C58: 0.1uF/16V, adafruit:CPOL-USR/2012-12R
- added C66, C76, C86: 1.0uF, resistor:C-USC0402
- added C68, C77, C87: 0.01uF, resistor:C-USC0402
- added L10, L11, L4, L5, L6, L7: 1000@100MHz, dp_devices:FERRITE-0402
- added L8: (no value), dp_devices:FERRITE-0402
- added MSATA, PCIE1, PCIE2: 679105700, con-molex:679105700
- added R18, R19, R20, R22: 2.2k, adafruit:R-US_M0805
- added R21: 1kΩ, adafruit:R-US_M0805
- added RT13, RT14, RT17, RT18, RT21, RT22: 20Ω, adafruit:R-US_M0805
- added RT15, RT16, RT19, RT20, RT23, RT24: 49.9Ω, adafruit:R-US_M0805
- added RT25, RT26, RT27: 4.7kΩ, adafruit:R-US_M0805
- added RT28: 1.6kΩ, adafruit:R-US_M0805
- added U$7: MCP1700T-1502E/TT, Microchip_By_element14_Batch_1:MCP1700T-1802E/TT
- added U7: XIO3130_ZHC_196, texas:XIO3130_ZHC_196
- X1: value 679105700 -> 5036-008-210-862; device con-molex:679105700 -> con-kyocera-elco:5036-008-210-862
Connections:
- removed net 3V2/NVCC_EIM0: ADC/DAC.VDDA, ADC/DAC.VDDIO, C12.-, C17.+, C23.-, C49.+, J1.P$63, J1.P$65, J1.P$67, J1.P$69, L2.2, L3.1, Q1.S, R14.1, R16.2, RT5.2, SD2_VSELECTG$1.Y1, SD2_VSELECTP.VCC, U$2.VIN, U$6.VIN, U1.FIX_PORT4, U1.SELFPWR, U1.VCC_D, U1.VCC_D_2, X1-2.S, X1-24.S, X1-39.S, X1-41.S, X1-52.S
- new net 12C3_SDA: GPIOB.3
- new net 1V5: C102.1, C104.1, C105.1, C106.1, C107.1, C108.1, C109.1, C110.1, C111.1, C112.1, C113.1, C114.1, C115.1, C116.1, C117.1, C118.1, C119.1, C120.1, C121.1, C122.1, C123.1, C124.1, C125.1, C126.1, C127.1, C52.+, C59.1, C69.1, C79.1, C89.1, L4.1, L5.1, L6.1, L7.1, L8.1, PCIE1-28.S, PCIE1-48.S, PCIE1-6.S, PCIE2-28.S, PCIE2-48.S, PCIE2-6.S, R18.2, U$7.VOUT, U7A.VDD15, U7A.VDD15_2, U7A.VDD15_3, U7A.VDD15_4, U7A.VDD15_5, U7A.VDD15_6, U7A.VDD15_7, U7A.VDD15_8, U7A.VDD15_9, U7B.RSVD, U7B.RSVD_3, U7B.VDD15, U7B.VDD15_10, U7B.VDD15_11, U7B.VDD15_12, U7B.VDD15_13, U7B.VDD15_14, U7B.VDD15_15, U7B.VDD15_16, U7B.VDD15_17, U7B.VDD15_18, U7B.VDD15_2, U7B.VDD15_3, U7B.VDD15_4, U7B.VDD15_5, U7B.VDD15_6, U7B.VDD15_7, U7B.VDD15_8, U7B.VDD15_9
- new net 3V2: ADC/DAC.VDDA, ADC/DAC.VDDIO, C100.1, C101.1, C12.-, C17.+, C23.-, C49.+, C51.+, C74.1, C84.1, C94.1, C95.1, C96.1, C97.1, C98.1, C99.1, GPIOA.1, GPIOB.1, J1.P$63, J1.P$65, J1.P$67, J1.P$69, L10.1, L11.1, L2.2, L3.1, MSATA-2.S, MSATA-24.S, MSATA-39.S, MSATA-41.S, MSATA-52.S, PCIE1-2.S, PCIE1-24.S, PCIE1-39.S, PCIE1-41.S, PCIE1-52.S, PCIE2-2.S, PCIE2-24.S, PCIE2-39.S, PCIE2-41.S, PCIE2-52.S, Q1.S, R14.1, R16.2, R19.1, R20.1, R21.2, R22.1, RT5.2, SD2_VSELECTG$1.Y1, SD2_VSELECTP.VCC, U$2.VIN, U$6.VIN, U$7.VIN, U1.FIX_PORT4, U1.SELFPWR, U1.VCC_D, U1.VCC_D_2, U4.VCC, U5.VCC, U6.VCC, U7A.RSVD, U7A.VDD33, U7A.VDD33_2, U7B.VDD33, U7B.VDD33_2, U7B.VDD33_3, U7B.VDD33_4, U7B.VDD33_5, U7B.VDD33_6
- new net DN1_PERST: PCIE1-22.S, RT27.2, U7A.*DN1_PERST
- new net DN2_PERST: PCIE2-22.S, RT25.2, U7A.*DN2_PERST
- new net DN3_PERST: RT26.2, U7A.*DN3_PERST
- new net N$62: C54.-, PCIE2-31.S
- new net N$63: C53.-, PCIE2-33.S
- new net N$66: C56.-, PCIE1-31.S
- new net N$67: C55.-, PCIE1-33.S
- new net N$75: C57.+, U7A.UP_REFCKIN
- new net N$77: C58.+, U7A.UP_REFCKIP
- new net N$79: GPIOB.12
- new net N$80: GPIOB.13
- new net PCIE_RXM1: PCIE1-23.S, U7A.DN1_PERN
- new net PCIE_RXM2: PCIE2-23.S, U7B.DN2_PERN
- new net PCIE_RXM3: U7B.DN3_PERN
- new net PCIE_RXP1: PCIE1-25.S, U7A.DN1_PERP
- new net PCIE_RXP2: PCIE2-25.S, U7B.DN2_PERP
- new net PCIE_RXP3: U7B.DN3_PERP
- new net PCIE_TXM1: C56.+, U7A.DN1_PETN
- new net PCIE_TXM2: C54.+, U7B.DN2_PETN
- new net PCIE_TXM3: U7B.DN3_PETN
- new net PCIE_TXP1: C55.+
- new net PCIE_TXP2: C53.+, U7B.DN2_PETP
- new net PCIE_TXP3: U7B.DN3_PETP
- new net REFCLKN_1: PCIE1-11.S, RT14.2, RT16.1
- new net REFCLKN_1_R: RT14.1, U7A.DN1_REFCK_ON
- new net REFCLKN_2: PCIE2-11.S, RT22.2, RT24.1
- new net REFCLKN_2_R: RT22.1, U7B.DN2_REFCKON
- new net REFCLKN_3: RT18.2, RT20.1
- new net REFCLKN_3_R: RT18.1, U7B.DN3_REFCKON
- new net REFCLKP_1: PCIE1-13.S, RT13.2, RT15.1
- new net REFCLKP_1_R: RT13.1, U7A.DN1_REFCK_OP
- new net REFCLKP_2: PCIE2-13.S, RT21.2, RT23.1
- new net REFCLKP_2_R: RT21.1, U7B.DN2_REFCKOP
- new net REFCLKP_3: RT17.2, RT19.1
- new net REFCLKP_3_R: RT17.1, U7B.DN3_REFCKOP
- new net RXD0: GPIOA.9, R20.2, U4.IN_A2
- new net RXD1: GPIOA.11, R19.2, U5.IN_A2
- new net RXD2: GPIOA.13, R22.2, U6.IN_A2
- new net TXD0: GPIOA.8, U4.OUT_Y1
- new net TXD1: GPIOA.10, U5.OUT_Y1
- new net TXD2: GPIOA.12, U6.OUT_Y1
- new net UIM_AUX1_1: X3.C6
- new net UIM_AUX1_2: X1.C6
- new net UIM_AUX2_1: X3.C8
- new net UIM_AUX2_2: X1.C8
- new net UIM_CLK_1: PCIE1-12.S, X3.C2
- new net UIM_CLK_2: PCIE2-12.S, X1.C2
- new net UIM_DATA_1: PCIE1-10.S, X3.C4
- new net UIM_DATA_2: PCIE2-10.S, X1.C4
- new net UIM_PWR_1: PCIE1-8.S, X3.C1
- new net UIM_PWR_2: PCIE2-8.S, X1.C1
- new net UIM_RST_1: PCIE1-14.S, X3.C5
- new net UIM_RST_2: PCIE2-14.S, X1.C5
- new net UIM_VPP_1: PCIE1-16.S, X3.C7
- new net UIM_VPP_2: PCIE2-16.S, X1.C7
- new net VAUX33REF: R21.1, U7A.VAUX33_REF
- new net VDD15REF: C103.1, L8.2, U7A.VDD15_REF
- new net VDD33REF: C85.1, L11.2, U7A.VDD33_REF
- new net VDDA15_0: C60.1, C61.1, C62.1, C63.1, L4.2, U7A.VDDA15_10, U7A.VDDA15_6, U7A.VDDA15_7, U7A.VDDA15_8, U7A.VDDA15_9
- new net VDDA15_1: C70.1, C71.1, C72.1, C73.1, L5.2, U7A.VDDA15_2, U7A.VDDA15_3, U7A.VDDA15_4, U7A.VDDA15_5
- new net VDDA15_2: C80.1, C81.1, C82.1, C83.1, L6.2, U7B.VDDA15, U7B.VDDA15_4, U7B.VDDA15_5, U7B.VDDA15_6, U7B.VDDA15_7
- new net VDDA15_3: C90.1, C91.1, C92.1, C93.1, L7.2, U7A.VDDA15, U7A.VDDA15_11, U7A.VDDA15_12, U7B.VDDA15_2, U7B.VDDA15_3
- new net VDDA33F: C75.1, L10.2, U7A.VDDA33
- new net VDDCOMB15: C86.1, C87.1, C88.1, U7A.VDD_COMB15
- new net VDDCOMB33: C76.1, C77.1, C78.1, U7A.VDD_COMB33
- new net VDDCOMBIO: C66.1, C67.1, C68.1, U7A.VDD_COMBIO
- net +5V: now also GPIOA.2, GPIOB.2
- net CLK1_N: now also C57.-
- net CLK1_P: now also C58.-
- net DISP1_DATA00: now also EXT_RADIO_INTERFACE.3
- net DISP1_DATA01: now also EXT_RADIO_INTERFACE.2
- net DISP1_DATA02: now also GPIOB.8
- net DISP1_DATA03: now also GPIOB.9
- net DISP1_DATA04: now also GPIOB.10
- net DISP1_DATA05: now also RT28.2, U7A.*UP_PERST
- net DISP1_DATA06: now also GPIOB.11
- net ECSPI2_MISO: now also GPIOA.4
- net ECSPI2_MOSI: now also GPIOA.3
- net ECSPI2_SCLK: now also GPIOA.5
- net ECSPI2_SS0: now also GPIOA.6
- net ECSPI2_SS1: now also GPIOA.7
- net I2C1_SCL: now also MSATA-30.S, U7B.SCL; no longer X1-30.S
- net I2C1_SDA: now also MSATA-32.S, U7B.SDA; no longer X1-32.S
- net I2C3_SCL: now also GPIOB.4
- net MSATA_DISABLE: now also MSATA-20.S, PCIE1-20.S, PCIE2-20.S; no longer X1-20.S
- net N$51: now also MSATA-23.S; no longer X1-23.S
- net N$59: now also MSATA-25.S; no longer X1-25.S
- net N$60: now also MSATA-31.S; no longer X1-31.S
- net N$61: now also MSATA-33.S; no longer X1-33.S
- net PCIE_RXM: now also U7A.UP_PERN
- net PCIE_RXP: now also U7A.UP_PERP
- net PCIE_TXM: now also U7A.UP_PETN
- net PCIE_TXP: now also U7A.DN1_PETP, U7A.UP_PETP
- net PE: now also C100.2, C101.2, C102.2, C103.2, C104.2, C105.2, C106.2, C107.2, C108.2, C109.2, C110.2, C111.2, C112.2, C113.2, C114.2, C115.2, C116.2, C117.2, C118.2, C119.2, C120.2, C121.2, C122.2, C123.2, C124.2, C125.2, C126.2, C127.2, C51.-, C52.-, C59.2, C60.2, C61.2, C62.2, C63.2, C66.2, C67.2, C68.2, C69.2, C70.2, C71.2, C72.2, C73.2, C74.2, C75.2, C76.2, C77.2, C78.2, C79.2, C80.2, C81.2, C82.2, C83.2, C84.2, C85.2, C86.2, C87.2, C88.2, C89.2, C90.2, C91.2, C92.2, C93.2, C94.2, C95.2, C96.2, C97.2, C98.2, C99.2, EXT_RADIO_INTERFACE.1, GPIOA.14, GPIOB.14, MSATA-15.S, MSATA-18.S, MSATA-21.S, MSATA-26.S, MSATA-27.S, MSATA-29.S, MSATA-34.S, MSATA-35.S, MSATA-37.S, MSATA-4.S, MSATA-40.S, MSATA-43.S, MSATA-50.S, MSATA-9.S, PCIE1-15.S, PCIE1-18.S, PCIE1-21.S, PCIE1-26.S, PCIE1-27.S, PCIE1-29.S, PCIE1-34.S, PCIE1-35.S, PCIE1-37.S, PCIE1-4.S, PCIE1-40.S, PCIE1-43.S, PCIE1-50.S, PCIE1-9.S, PCIE2-15.S, PCIE2-18.S, PCIE2-21.S, PCIE2-26.S, PCIE2-27.S, PCIE2-29.S, PCIE2-34.S, PCIE2-35.S, PCIE2-37.S, PCIE2-4.S, PCIE2-40.S, PCIE2-43.S, PCIE2-50.S, PCIE2-9.S, R18.1, RT15.2, RT16.2, RT19.2, RT20.2, RT23.2, RT24.2, RT25.1, RT26.1, RT27.1, RT28.1, U$7.GND, U4.GND, U5.GND, U6.GND, U7A.RSVD_2, U7A.VSS, U7A.VSSA, U7A.VSSA_2, U7A.VSSA_3, U7A.VSSA_4, U7A.VSSA_5, U7A.VSSA_6, U7A.VSSA_7, U7A.VSSA_REF, U7A.VSSD_REF, U7A.VSS_10, U7A.VSS_11, U7A.VSS_12, U7A.VSS_13, U7A.VSS_14, U7A.VSS_15, U7A.VSS_16, U7A.VSS_17, U7A.VSS_18, U7A.VSS_19, U7A.VSS_2, U7A.VSS_20, U7A.VSS_21, U7A.VSS_22, U7A.VSS_23, U7A.VSS_24, U7A.VSS_25, U7A.VSS_26, U7A.VSS_27, U7A.VSS_28, U7A.VSS_29, U7A.VSS_3, U7A.VSS_30, U7A.VSS_31, U7A.VSS_32, U7A.VSS_33, U7A.VSS_34, U7A.VSS_35, U7A.VSS_4, U7A.VSS_5, U7A.VSS_6, U7A.VSS_7, U7A.VSS_8, U7A.VSS_9, U7B.DN1_DPSTRP, U7B.DN2_DPSTRP, U7B.DN3_DPSTRP, U7B.RSVD_2, U7B.VSS, U7B.VSSA, U7B.VSSA_10, U7B.VSSA_11, U7B.VSSA_12, U7B.VSSA_13, U7B.VSSA_14, U7B.VSSA_15, U7B.VSSA_2, U7B.VSSA_3, U7B.VSSA_4, U7B.VSSA_5, U7B.VSSA_6, U7B.VSSA_7, U7B.VSSA_8, U7B.VSSA_9, U7B.VSS_10, U7B.VSS_11, U7B.VSS_12, U7B.VSS_13, U7B.VSS_14, U7B.VSS_2, U7B.VSS_3, U7B.VSS_4, U7B.VSS_5, U7B.VSS_6, U7B.VSS_7, U7B.VSS_8, U7B.VSS_9, X1.C3, X3.C3; no longer X1-15.S, X1-18.S, X1-21.S, X1-26.S, X1-27.S, X1-29.S, X1-34.S, X1-35.S, X1-37.S, X1-4.S, X1-40.S, X1-43.S, X1-50.S, X1-9.S
- net POR_B: now also MSATA-22.S; no longer X1-22.S
- net SD3_CLK: now also GPIOB.6
- net SD3_CMD: now also GPIOB.7
- net UART1_RX_DATA: now also U4.OUT_Y2
- net UART1_TX_DATA: now also U4.IN_A1
- net UART2_RX_DATA: now also U5.OUT_Y2
- net UART2_TX_DATA: now also U5.IN_A1
- net UART3_RX_DATA: now also U6.OUT_Y2
- net UART3_TX_DATA: now also U6.IN_A1
- net USB_OTG_ID: now also GPIOB.5
- net V_1V5: now also MSATA-28.S, MSATA-48.S, MSATA-6.S; no longer X1-28.S, X1-48.S, X1-6.S
Other:
- note added: "1x stacked USB and HDMI Digital Coax S/PDIF LEDS Various Display connectors (Maybe leave off) RTC battery HEader MIPI CSI connector?"
- note added: "Main Power feeds are +5V and 3V2"
- note removed: "1x stacked USB and HDMI IR? Digital Coax S/PDIF LEDS Various Display connectors (Maybe leave off) RTC battery HEader MIPI CSI connector?"
- note removed: "Main Power feeds are +5V and 3V2/NVCC_EIM0"
- moved on the sheet: GPIOA, GPIOB, U4, U5, U6, X3
