File: Rasberry Pi based Cellphone/Main Schematic.sch (EAGLE design)
At the start: 239 parts, among them IC1 PCM2904DB, J1 Main B2B Header, J2 Second B2B Header, J3 Third B2B Header, Q1 20V P-Channel Mosfet, SW1 SPST_TACT-KMR2, SW2 SPST_TACT-KMR2, SW3 SPST_TACT-KMR2, U7 XIO3130_ZHC_196, X1 5036-008-210-862, X3 5036-008-210-862

Commit message: fixed some errors in schematic and made brd easier to look at
Parts:
- C1: value (none) -> 1uF
- C3, C49: value (none) -> 10uF/6.3V
- D3: value (none) -> RB521CS-30
- L8: value (none) -> 1000@100MHz
- Q2: value (none) -> 12MHz
- UART_BUF_0, UART_BUF_1, UART_BUF_2: value (none) -> NLX2G16
- USBCON_1: value (none) -> USB_1
- USBCON_OTG: value (none) -> USB_OTG
- USB_CURR_LIM: value (none) -> MIC2026-1YM
- USB_HUB: value (none) -> USB Hub
- VREG_1: value (none) -> +5V -> 3V2
- renumbered IC1 to USB_AUDIO_CODEC, U1 to USB_HUB, U2 to VREG_1, U3 to USB_CURR_LIM, U4 to UART_BUF_0, U5 to UART_BUF_1, U6 to UART_BUF_2, X5 to USBCON_OTG, X6 to USBCON_1
Connections:
- net VCC_1V8 renamed 1V8
- new net LVDS0_TX2_P: J2.P$74
- net AUD5_TXD: now also J2.P$53
- net PE: now also J2.P$12
- net USB_HUB_DN2: now also PCIE1-36.S
- net USB_HUB_DN3: now also PCIE2-36.S
- net USB_HUB_DP2: now also PCIE1-38.S
- net USB_HUB_DP3: now also PCIE2-38.S
Other:
- moved on the sheet: ON/OFF?, RT15, RT16, RT19, RT20, RT23, RT24
